File: Hardware/sparkfun-mlx90640-qwiic-breakout.brd (EAGLE design)
At the start: 25.4 x 25.4 mm, 38 parts, among them J2 SMD, J3 PTH, J4 SMD, U1 MLX90640

Commit message: updating to reds
Parts:
- removed U$15: (no value), buzzard_labels:55X35#____3
- removed U$17: (no value), buzzard_labels:110X75#____4
- removed U$3: SPARKX-LOGO4, SparkX:SPARKX-MEDIUM
- added LOGO2: SFE_LOGO_NAME_FLAME.1_INCH, SparkFun-Aesthetics:SFE_LOGO_NAME_FLAME_.1
- added LOGO3: SFE_LOGO_NAME.1_INCH, SparkFun-Aesthetics:SFE_LOGO_NAME_.1
- added LOGO4: REVISION, SparkFun-Aesthetics:REVISION
- J2, J4: value SMD -> (none); device SparkX:1X04_1MM_RA -> SparkFun-Connectors:1X04_1MM_RA
- U$2: value SPARKX-LOGO5 -> (none); device SparkX:SPARKX-LARGE -> buzzard_labels (12):110X75#____0
- U1: value MLX90640 -> 110DEG; device MLX90540:MLX90640 -> SparkFun-IC-Special-Function:MLX90540_MLX90640
- moved FRAME1 12.8 mm to (-10.2, -7.62)
- moved U$2 8.43 mm to (19.4, 17.8), flipped to the top
Other:
- board text added: "Andy England"
- board text added: "v01"
- board text removed: "X01"
Changed lines of the file:
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@@
 <drawing>
 <settings>
-<setting alwaysvectorfont="yes"/>
+<setting alwaysvectorfont="no"/>
 <setting verticaltext="up"/>
 </settings>
-<grid distance="0.05" unitdist="inch" unit="inch" style="lines" multiple="1" display="yes" altdistance="0.005" altunitdist="inch" altunit="inch"/>
+<grid distance="1.23" unitdist="mm" unit="mm" style="lines" multiple="1" display="yes" altdistance="0.005" altunitdist="inch" altunit="inch"/>
 <layers>
 <layer number="1" name="Top" color="4" fill="1" visible="yes" active="yes"/>
@@
 <wire x1="25.4" y1="25.4" x2="0" y2="25.4" width="0.1524" layer="20"/>
 <wire x1="0" y1="25.4" x2="0" y2="0" width="0.1524" layer="20"/>
-<text x="22.86" y="19.2405" size="1.27" layer="16" font="vector" ratio="15" rot="MR0" align="bottom-center">X01</text>
-<text x="34.29" y="-8.89" size="1.27" layer="51" font="vector" ratio="15" align="bottom-center">Jim Lindblom</text>
+<text x="25.2095" y="6.35" size="1.27" layer="16" font="vector" ratio="15" rot="SMR270" align="bottom-center">v01</text>
+<text x="24.13" y="-7.62" size="1.778" layer="51" font="vector" align="bottom-center">Jim Lindblom</text>
+<text x="22.86" y="-10.16" size="1.778" layer="51" font="vector" align="bottom-center">Andy England</text>
 </plain>
 <attributes>
@@
 <attribute name="PROD_ID" value="DIO-00819" x="2.54" y="6.9215" size="1.778" layer="27" display="off"/>
 </element>
-<element name="FRAME1" library="SparkFun-Aesthetics" package="CREATIVE_COMMONS" value="FRAME-LETTER" x="2.54" y="-8.89"/>
-<element name="J2" library="SparkX" package="1X04_1MM_RA" value="SMD" x="20.32" y="12.7" rot="R90"/>
+<element name="FRAME1" library="SparkFun-Aesthetics" package="CREATIVE_COMMONS" value="FRAME-LETTER" x="-10.16" y="-7.62"/>
+<element name="J2" library="SparkFun-Connectors" package="1X04_1MM_RA" value="" x="20.32" y="12.7" rot="R90">
+<attribute name="PROD_ID" value="CONN-13694" x="20.32" y="12.7" size="1.778" layer="27" rot="R90" display="off"/>
+<attribute name="VALUE" value="" x="20.32" y="12.7" size="1.778" layer="27" rot="R90" display="off"/>
+</element>
 <element name="J3" library="SparkX" package="1X04_NO_SILK" value="PTH" x="8.89" y="1.27"/>
-<element name="J4" library="SparkX" package="1X04_1MM_RA" value="SMD" x="5.08" y="12.7" rot="R270"/>
+<element name="J4" library="SparkFun-Connectors" package="1X04_1MM_RA" value="" x="5.08" y="12.7" rot="R270">
+<attribute name="PROD_ID" value="CONN-13694" x="5.08" y="12.7" size="1.778" layer="27" rot="R270" display="off"/>
+<attribute name="VALUE" value="" x="5.08" y="12.7" size="1.778" layer="27" rot="R270" display="off"/>
+</element>
 <element name="JP1" library="SparkFun-Jumpers" package="SMT-JUMPER_3_2-NC_TRACE_NO-SILK" value="I2C" x="19.05" y="7.62" rot="MR0"/>
 <element name="R1" library="SparkFun-Resistors" package="0603" value="2.2k" x="17.78" y="7.62" rot="R90">
@@
 <attribute name="PROD_ID" value="RES-07856" x="2.54" y="8.255" size="1.778" layer="27" display="off"/>
 </element>
-<element name="U1" library="MLX90540" package="MLX90640" value="MLX90640" x="12.7" y="12.7" rot="R90"/>
+<element name="U1" library="SparkFun-IC-Special-Function" package="MLX90540_MLX90640" value="110DEG" x="12.7" y="12.7" rot="R90">
+<attribute name="PROD_ID" value="IC-14041" x="12.7" y="12.7" size="1.778" layer="27" rot="R90" display="off"/>
+<attribute name="VALUE" value="110DEG" x="12.7" y="12.7" size="1.778" layer="27" rot="R90" display="off"/>
+</element>
 <element name="JP3" library="SparkFun" package="STAND-OFF" value="STAND-OFF" x="2.54" y="22.86"/>
 <element name="JP4" library="SparkFun" package="STAND-OFF" value="STAND-OFF" x="22.86" y="22.86"/>
 <element name="JP2" library="SparkFun" package="MICRO-FIDUCIAL" value="FIDUCIALUFIDUCIAL" x="24.765" y="0.635"/>
 <element name="JP6" library="SparkFun" package="MICRO-FIDUCIAL" value="FIDUCIALUFIDUCIAL" x="24.765" y="0.635" rot="MR0"/>
-<element name="U$2" library="SparkX" package="SPARKX-LARGE" value="SPARKX-LOGO5" x="12.7" y="22.86" rot="MR0"/>
 <element name="LOGO1" library="SparkFun-Aesthetics" package="OSHW-LOGO-MINI" value="OSHW-LOGOMINI" x="22.86" y="6.35" rot="MR0"/>
-<element name="U$3" library="SparkX" package="SPARKX-MEDIUM" value="SPARKX-LOGO4" x="12.7" y="22.86"/>
 <element name="JP5" library="SparkFun" package="MICRO-FIDUCIAL" value="FIDUCIALUFIDUCIAL" x="0.635" y="24.765"/>
 <element name="JP7" library="SparkFun" package="MICRO-FIDUCIAL" value="FIDUCIALUFIDUCIAL" x="0.635" y="24.765" rot="MR0"/>
@@
 <element name="U$14" library="buzzard_labels" package="QWIIC_IR_ARRAY0" value="" x="5.334" y="20.6375"/>
 <element name="U$16" library="Labels" package="I_SUPER2_C-()-03" value="" x="20.5105" y="6.223" rot="MR0"/>
-<element name="U$15" library="buzzard_labels" package="55X35#____3" value="" x="19.3802" y="19.05"/>
-<element name="U$17" library="buzzard_labels" package="110X75#____4" value="" x="19.05" y="17.145"/>
+<element name="LOGO2" library="SparkFun-Aesthetics" package="SFE_LOGO_NAME_FLAME_.1" value="SFE_LOGO_NAME_FLAME.1_INCH" x="18.669" y="19.685" rot="MR0"/>
+<element name="LOGO4" library="SparkFun-Aesthetics" package="REVISION" value="REVISION" x="1.27" y="-10.16"/>
+<element name="LOGO3" library="SparkFun-Aesthetics" package="SFE_LOGO_NAME_.1" value="SFE_LOGO_NAME.1_INCH" x="6.731" y="21.082"/>
+<element name="U$2" library="buzzard_labels (12)" package="110X75#____0" value="" x="19.431" y="17.78"/>
 </elements>
 <signals>

Commit message: Post design review changes
Routing:
- net SDA: track 30.4 -> 32.0 mm
- net SCL: track 32.6 -> 33.5 mm
Other:
- board text added: "Units in In."
- board text added: "v10"
- board text removed: "v01"
Changed lines of the file:
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@@
 <?xml version="1.0" encoding="utf-8"?>
 <!DOCTYPE eagle SYSTEM "eagle.dtd">
-<eagle version="9.0.1">
+<eagle version="9.1.0">
 <drawing>
 <settings>
@@
 <layer number="45" name="Holes" color="7" fill="1" visible="yes" active="yes"/>
 <layer number="46" name="Milling" color="3" fill="1" visible="no" active="yes"/>
-<layer number="47" name="Measures" color="7" fill="1" visible="no" active="yes"/>
+<layer number="47" name="Measures" color="7" fill="1" visible="yes" active="yes"/>
 <layer number="48" name="Document" color="7" fill="1" visible="no" active="yes"/>
 <layer number="49" name="Reference" color="7" fill="1" visible="no" active="yes"/>
@@
 <wire x1="25.4" y1="25.4" x2="0" y2="25.4" width="0.1524" layer="20"/>
 <wire x1="0" y1="25.4" x2="0" y2="0" width="0.1524" layer="20"/>
-<text x="25.2095" y="6.35" size="1.27" layer="16" font="vector" ratio="15" rot="SMR270" align="bottom-center">v01</text>
+<text x="25.2095" y="6.35" size="1.27" layer="16" font="vector" ratio="15" rot="SMR270" align="bottom-center">v10</text>
 <text x="24.13" y="-7.62" size="1.778" layer="51" font="vector" align="bottom-center">Jim Lindblom</text>
 <text x="22.86" y="-10.16" size="1.778" layer="51" font="vector" align="bottom-center">Andy England</text>
+<dimension x1="2.54" y1="22.86" x2="2.54" y2="2.54" x3="-1.23" y3="12.7" textsize="1.778" layer="47" unit="inch"/>
+<dimension x1="0" y1="0" x2="0" y2="25.4" x3="-4.92" y3="12.7" textsize="1.778" layer="47" unit="inch"/>
+<dimension x1="0" y1="25.4" x2="25.4" y2="25.4" x3="12.7" y3="30.75" textsize="1.778" layer="47" unit="inch"/>
+<dimension x1="2.54" y1="22.86" x2="22.86" y2="22.86" x3="12.7" y3="27.06" textsize="1.778" layer="47" unit="inch"/>
+<text x="-13.53" y="25.83" size="1.778" layer="47" font="vector">Units in In.</text>
 </plain>
 <attributes>
@@
 <param name="checkStop" value="0"/>
 <param name="checkValues" value="0"/>
+<param name="checkNames" value="1"/>
+<param name="checkWireStubs" value="1"/>
+<param name="checkPolygonWidth" value="0"/>
 <param name="useDiameter" value="13"/>
 <param name="maxErrors" value="50"/>
@@
 <via x="18.6055" y="13.97" extent="1-16" drill="0.3048"/>
 <wire x1="11.28" y1="11.2" x2="12.7" y2="9.78" width="0.1524" layer="16"/>
-<wire x1="18.6055" y1="13.97" x2="16.51" y2="11.8745" width="0.1524" layer="16"/>
-<wire x1="16.51" y1="11.8745" x2="16.51" y2="10.16" width="0.1524" layer="16"/>
-<wire x1="16.51" y1="10.16" x2="15.24" y2="8.89" width="0.1524" layer="16"/>
+<wire x1="16.51" y1="11.8745" x2="18.6055" y2="13.97" width="0.1524" layer="16"/>
 <wire x1="13.59" y1="8.89" x2="12.7" y2="9.78" width="0.1524" layer="16"/>
 <wire x1="15.24" y1="8.89" x2="13.59" y2="8.89" width="0.1524" layer="16"/>
@@
 <via x="19.05" y="5.08" extent="1-16" drill="0.3048"/>
 <wire x1="17.78" y1="3.81" x2="19.05" y2="5.08" width="0.1524" layer="16"/>
-<wire x1="19.05" y1="5.08" x2="19.05" y2="5.5" width="0.1524" layer="1"/>
-<wire x1="19.05" y1="5.5" x2="20.32" y2="6.77" width="0.1524" layer="1"/>
 <wire x1="15.24" y1="8.89" x2="15.24" y2="6.35" width="0.1524" layer="16"/>
 <wire x1="15.24" y1="6.35" x2="17.78" y2="3.81" width="0.1524" layer="16"/>
+<wire x1="15.24" y1="8.89" x2="16.002" y2="8.89" width="0.1524" layer="16"/>
+<wire x1="16.002" y1="8.89" x2="16.51" y2="9.398" width="0.1524" layer="16"/>
+<wire x1="16.51" y1="9.398" x2="16.51" y2="11.8745" width="0.1524" layer="16"/>
+<wire x1="19.05" y1="5.08" x2="19.812" y2="5.08" width="0.1524" layer="1"/>
+<wire x1="19.812" y1="5.08" x2="20.32" y2="5.588" width="0.1524" layer="1"/>
+<wire x1="20.32" y1="5.588" x2="20.32" y2="6.77" width="0.1524" layer="1"/>
 </signal>
 <signal name="SDA">
@@
 <wire x1="15.121" y1="12.2" x2="15.8115" y2="12.8905" width="0.1524" layer="16"/>
 <wire x1="14.764753125" y1="10.635246875" x2="14.764753125" y2="9.785246875" width="0.1524" layer="1"/>
-<wire x1="14.764753125" y1="9.785246875" x2="16.085" y2="8.465" width="0.1524" layer="1"/>
-<wire x1="16.085" y1="8.465" x2="17.78" y2="6.77" width="0.1524" layer="1"/>
 <wire x1="14.764753125" y1="10.635246875" x2="14.764753125" y2="12.2" width="0.1524" layer="16"/>
-<wire x1="13.97" y1="1.27" x2="13.97" y2="6.35" width="0.1524" layer="1"/>
-<wire x1="13.97" y1="6.35" x2="16.085" y2="8.465" width="0.1524" layer="1"/>
+<wire x1="13.97" y1="1.27" x2="13.97" y2="6.15" width="0.1524" layer="1"/>
+<wire x1="13.97" y1="6.15" x2="13.97" y2="6.35" width="0.1524" layer="1"/>
+<wire x1="17.78" y1="6.77" x2="15.99" y2="6.77" width="0.1524" layer="1"/>
+<wire x1="15.99" y1="6.77" x2="15.37" y2="6.77" width="0.1524" layer="1"/>
+<wire x1="14.764753125" y1="7.384753125" x2="14.76" y2="7.38" width="0.1524" layer="1"/>
+<wire x1="14.764753125" y1="7.384753125" x2="14.764753125" y2="10.635246875" width="0.1524" layer="1"/>
+<wire x1="13.97" y1="6.15" x2="13.97" y2="6.35" width="0.1524" layer="1"/>
+<wire x1="13.97" y1="6.35" x2="13.97" y2="6.15" width="0.1524" layer="1"/>
+<wire x1="15.99" y1="6.77" x2="14.76" y2="6.77" width="0.1524" layer="1"/>
+<wire x1="14.76" y1="6.77" x2="14.39" y2="6.77" width="0.1524" layer="1"/>
+<wire x1="14.39" y1="6.77" x2="13.97" y2="6.35" width="0.1524" layer="1"/>
+<wire x1="14.764753125" y1="7.384753125" x2="14.764753125" y2="6.774753125" width="0.1524" layer="1"/>
+<wire x1="14.764753125" y1="6.774753125" x2="14.76" y2="6.77" width="0.1524" layer="1"/>
 </signal>
 <signal name="N$1">
@@
 </signal>
 </signals>
+<mfgpreviewcolors>
+<mfgpreviewcolor name="soldermaskcolor" color="0xC8008000"/>
+<mfgpreviewcolor name="silkscreencolor" color="0xFFFEFEFE"/>
+<mfgpreviewcolor name="backgroundcolor" color="0xFF282828"/>
+<mfgpreviewcolor name="coppercolor" color="0xFFFFBF00"/>
+<mfgpreviewcolor name="substratecolor" color="0xFF786E46"/>
+</mfgpreviewcolors>
 <errors>
 </errors>

Commit message: fixing issues
Routing:
- net SDA: track 32.0 -> 30.2 mm
