File: Hardware/sparkfun-mlx90640-qwiic-breakout.brd (EAGLE design)
At the start: 25.4 x 25.4 mm, 39 parts, among them J3 PTH, U1 110DEG

Commit message: pulling in PTH holes, needs repanel
Parts:
- J2, J4: device SparkFun-Connectors:1X04_1MM_RA -> SparkFun-Connectors:JST04_1MM_RA
- moved LOGO3 6.23 mm to (12.7, 22.9)
- moved LOGO2 6.13 mm to (12.7, 21.1)
Other:
- board text added: "v13"
- board text removed: "v12"
Changed lines of the file:
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@@
 <?xml version="1.0" encoding="utf-8"?>
 <!DOCTYPE eagle SYSTEM "eagle.dtd">
-<eagle version="9.0.1">
+<eagle version="9.1.0">
 <drawing>
 <settings>
@@
 <layer number="115" name="ReferenceISLANDS" color="7" fill="1" visible="no" active="no"/>
 <layer number="116" name="Patch_BOT" color="9" fill="4" visible="no" active="no"/>
+<layer number="117" name="PM_Ref" color="26" fill="1" visible="yes" active="yes"/>
 <layer number="118" name="Rect_Pads" color="7" fill="1" visible="no" active="no"/>
+<layer number="119" name="PF_Ref" color="31" fill="1" visible="yes" active="yes"/>
+<layer number="120" name="WFL_Ref" color="25" fill="1" visible="yes" active="yes"/>
 <layer number="121" name="_tsilk" color="7" fill="1" visible="no" active="no"/>
 <layer number="122" name="_bsilk" color="7" fill="1" visible="no" active="no"/>
@@
 <wire x1="25.4" y1="25.4" x2="0" y2="25.4" width="0.1524" layer="20"/>
 <wire x1="0" y1="25.4" x2="0" y2="0" width="0.1524" layer="20"/>
-<text x="25.2095" y="6.35" size="1.27" layer="16" font="vector" ratio="15" rot="SMR270" align="bottom-center">v12</text>
+<text x="25.2095" y="6.35" size="1.27" layer="16" font="vector" ratio="15" rot="SMR270" align="bottom-center">v13</text>
 <text x="24.13" y="-7.62" size="1.778" layer="51" font="vector" align="bottom-center">Jim Lindblom</text>
 <text x="22.86" y="-10.16" size="1.778" layer="51" font="vector" align="bottom-center">Andy England</text>
@@
 <param name="checkStop" value="0"/>
 <param name="checkValues" value="0"/>
+<param name="checkNames" value="1"/>
+<param name="checkWireStubs" value="1"/>
+<param name="checkPolygonWidth" value="0"/>
 <param name="useDiameter" value="13"/>
 <param name="maxErrors" value="50"/>
@@
 <attribute name="PROD_ID" value="DIO-00819" x="2.54" y="6.9215" size="1.778" layer="27" display="off"/>
 </element>
-<element name="FRAME1" library="SparkFun-Aesthetics" package="CREATIVE_COMMONS" value="FRAME-LETTER" x="-10.16" y="-7.62"/>
-<element name="J2" library="SparkFun-Connectors" package="1X04_1MM_RA" value="" x="20.32" y="12.7" rot="R90">
+<element name="FRAME1" library="SparkFun-Aesthetics" package="CREATIVE_COMMONS" value="FRAME-LETTER" x="-10.16" y="-7.62">
+<attribute name="DESIGNER" value="" x="-10.16" y="-7.62" size="1.778" layer="27" display="off"/>
+<attribute name="REV" value="" x="-10.16" y="-7.62" size="1.778" layer="27" display="off"/>
+</element>
+<element name="J2" library="SparkFun-Connectors" package="JST04_1MM_RA" value="" x="20.32" y="12.7" rot="R90">
 <attribute name="PROD_ID" value="CONN-13694" x="20.32" y="12.7" size="1.778" layer="27" rot="R90" display="off"/>
 <attribute name="VALUE" value="" x="20.32" y="12.7" size="1.778" layer="27" rot="R90" display="off"/>
 </element>
 <element name="J3" library="SparkX" package="1X04_NO_SILK" value="PTH" x="8.89" y="1.27"/>
-<element name="J4" library="SparkFun-Connectors" package="1X04_1MM_RA" value="" x="5.08" y="12.7" rot="R270">
+<element name="J4" library="SparkFun-Connectors" package="JST04_1MM_RA" value="" x="5.08" y="12.7" rot="R270">
 <attribute name="PROD_ID" value="CONN-13694" x="5.08" y="12.7" size="1.778" layer="27" rot="R270" display="off"/>
 <attribute name="VALUE" value="" x="5.08" y="12.7" size="1.778" layer="27" rot="R270" display="off"/>
@@
 <element name="U$14" library="buzzard_labels" package="QWIIC_IR_ARRAY0" value="" x="5.334" y="20.6375"/>
 <element name="U$16" library="Labels" package="I_SUPER2_C-()-03" value="" x="20.5105" y="6.223" rot="MR0"/>
-<element name="LOGO2" library="SparkFun-Aesthetics" package="SFE_LOGO_NAME_FLAME_.1" value="SFE_LOGO_NAME_FLAME.1_INCH" x="18.669" y="19.685" rot="MR0"/>
+<element name="LOGO2" library="SparkFun-Aesthetics" package="SFE_LOGO_NAME_FLAME_.1" value="SFE_LOGO_NAME_FLAME.1_INCH" x="12.7" y="21.082" rot="MR0"/>
 <element name="LOGO4" library="SparkFun-Aesthetics" package="REVISION" value="REVISION" x="1.27" y="-10.16"/>
-<element name="LOGO3" library="SparkFun-Aesthetics" package="SFE_LOGO_NAME_.1" value="SFE_LOGO_NAME.1_INCH" x="6.731" y="21.082"/>
+<element name="LOGO3" library="SparkFun-Aesthetics" package="SFE_LOGO_NAME_.1" value="SFE_LOGO_NAME.1_INCH" x="12.7" y="22.86"/>
 <element name="U$3" library="buzzard_labels (9)" package="55X35#1" value="" x="18.923" y="18.796"/>
 <element name="U$15" library="buzzard_labels (9)" package="110X75#0" value="" x="18.542" y="17.145"/>
@@
 <wire x1="16.51" y1="2.54" x2="17.78" y2="3.81" width="0.2032" layer="16"/>
 <via x="19.05" y="5.08" extent="1-16" drill="0.381"/>
-<wire x1="17.78" y1="3.81" x2="19.05" y2="5.08" width="0.1524" layer="16"/>
 <wire x1="15.24" y1="7.62" x2="15.24" y2="6.35" width="0.2032" layer="16"/>
 <wire x1="15.24" y1="6.35" x2="17.78" y2="3.81" width="0.2032" layer="16"/>
@@
 <wire x1="15.24" y1="7.62" x2="13.964909375" y2="7.62" width="0.2032" layer="16"/>
 <wire x1="13.964909375" y1="7.62" x2="11.5825875" y2="10.002321875" width="0.2032" layer="16"/>
+<wire x1="17.78" y1="3.81" x2="19.05" y2="5.08" width="0.2032" layer="16"/>
 </signal>
 <signal name="SDA">
@@
 </signal>
 </signals>
+<mfgpreviewcolors>
+<mfgpreviewcolor name="soldermaskcolor" color="0xC8008000"/>
+<mfgpreviewcolor name="silkscreencolor" color="0xFFFEFEFE"/>
+<mfgpreviewcolor name="backgroundcolor" color="0xFF282828"/>
+<mfgpreviewcolor name="coppercolor" color="0xFFFFBF00"/>
+<mfgpreviewcolor name="substratecolor" color="0xFF786E46"/>
+</mfgpreviewcolors>
 <errors>
 </errors>
