File: Hardware/sparkfun-mlx90640-qwiic-breakout.sch (EAGLE design)
At the start: 23 parts, among them J2 SMD, J3 PTH, J4 SMD, U1 MLX90640

Commit message: updating to reds
Parts:
- removed U$2: SPARKX-LOGO5, SparkX:SPARKX-LOGO5
- removed U$3: SPARKX-LOGO4, SparkX:SPARKX-LOGO4
- added LOGO2: SFE_LOGO_NAME_FLAME.1_INCH, SparkFun-Aesthetics:SFE_LOGO_NAME_FLAME.1_INCH
- added LOGO3: SFE_LOGO_NAME.1_INCH, SparkFun-Aesthetics:SFE_LOGO_NAME.1_INCH
- added LOGO4: REVISION, SparkFun-Aesthetics:REVISION
- J2, J4: value SMD -> (none); device SparkX:I2C_STANDARDJS-1MM -> SparkFun-Connectors:QWIIC_CONNECTORJS-1MM
- U1: value MLX90640 -> 110DEG; device MLX90540:MLX90640 -> SparkFun-IC-Special-Function:MLX90540_MLX906404
Connections:
- net 3.3V: now also J2.2, J4.2; no longer J2.VCC, J4.VCC
- net GND: now also J2.1, J4.1; no longer J2.GND, J4.GND
- net SCL: now also J2.4, J4.4; no longer J2.SCL, J4.SCL
- net SDA: now also J2.3, J4.3; no longer J2.SDA, J4.SDA
Other:
- note added: "Andy England"
- note added: "MLX90640"
- note added: "Qwiic/I2C Conections"
- note added: "v01"
Changed lines of the file:
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@@
 <drawing>
 <settings>
-<setting alwaysvectorfont="yes"/>
+<setting alwaysvectorfont="no"/>
 <setting verticaltext="up"/>
 </settings>
@@
 <parts>
 <part name="FRAME1" library="SparkFun-Aesthetics" deviceset="FRAME-LETTER" device=""/>
-<part name="U1" library="MLX90540" deviceset="MLX90640" device=""/>
+<part name="U1" library="SparkFun-IC-Special-Function" deviceset="MLX90540_MLX90640" device="" technology="4" value="110DEG"/>
 <part name="C1" library="SparkFun-Capacitors" deviceset="0.1UF" device="-0603-25V-(+80/-20%)" value="0.1uF"/>
 <part name="SUPPLY1" library="SparkFun-PowerSymbols" deviceset="3.3V" device=""/>
@@
 <part name="GND3" library="SparkFun-PowerSymbols" deviceset="GND" device=""/>
 <part name="SUPPLY4" library="SparkFun-PowerSymbols" deviceset="3.3V" device=""/>
-<part name="J2" library="SparkX" deviceset="I2C_STANDARD" device="JS-1MM" value="SMD"/>
+<part name="J2" library="SparkFun-Connectors" deviceset="QWIIC_CONNECTOR" device="JS-1MM"/>
 <part name="GND6" library="SparkFun" deviceset="GND" device=""/>
 <part name="SUPPLY7" library="SparkFun-PowerSymbols" deviceset="3.3V" device=""/>
@@
 <part name="GND7" library="SparkFun" deviceset="GND" device=""/>
 <part name="SUPPLY8" library="SparkFun-PowerSymbols" deviceset="3.3V" device=""/>
-<part name="J4" library="SparkX" deviceset="I2C_STANDARD" device="JS-1MM" value="SMD"/>
+<part name="J4" library="SparkFun-Connectors" deviceset="QWIIC_CONNECTOR" device="JS-1MM"/>
 <part name="GND8" library="SparkFun" deviceset="GND" device=""/>
 <part name="R1" library="SparkFun-Resistors" deviceset="2.2KOHM" device="-0603-1/10W-1%" value="2.2k"/>
@@
 <part name="JP2" library="SparkFun" deviceset="FIDUCIAL" device="UFIDUCIAL"/>
 <part name="JP6" library="SparkFun" deviceset="FIDUCIAL" device="UFIDUCIAL"/>
-<part name="U$2" library="SparkX" deviceset="SPARKX-LOGO" device="5" value="SPARKX-LOGO5"/>
 <part name="LOGO1" library="SparkFun-Aesthetics" deviceset="OSHW-LOGO" device="MINI"/>
-<part name="U$3" library="SparkX" deviceset="SPARKX-LOGO" device="4"/>
 <part name="JP5" library="SparkFun" deviceset="FIDUCIAL" device="UFIDUCIAL"/>
 <part name="JP7" library="SparkFun" deviceset="FIDUCIAL" device="UFIDUCIAL"/>
 <part name="JP8" library="SparkFun" deviceset="STAND-OFF" device=""/>
 <part name="JP9" library="SparkFun" deviceset="STAND-OFF" device=""/>
+<part name="LOGO2" library="SparkFun-Aesthetics" deviceset="SFE_LOGO_NAME_FLAME" device=".1_INCH"/>
+<part name="LOGO4" library="SparkFun-Aesthetics" deviceset="REVISION" device=""/>
+<part name="LOGO3" library="SparkFun-Aesthetics" deviceset="SFE_LOGO_NAME" device=".1_INCH"/>
 </parts>
 <sheets>
@@
 <text x="165.354" y="11.43" size="2.54" layer="94">Jim Lindblom</text>
 <text x="106.68" y="93.98" size="1.778" layer="97">7-bit unshifted I2C Address: 0x33</text>
+<text x="236.22" y="7.62" size="2.54" layer="94" font="vector">v01</text>
+<text x="168.656" y="7.366" size="2.54" layer="94" font="vector">Andy England</text>
+<text x="114.3" y="132.08" size="2.54" layer="95" font="vector">MLX90640</text>
+<text x="50.8" y="63.5" size="2.54" layer="95" font="vector">Qwiic/I2C Conections</text>
 </plain>
 <instances>
@@
 <instance part="JP2" gate="G$1" x="233.68" y="27.94"/>
 <instance part="JP6" gate="G$1" x="236.22" y="27.94"/>
-<instance part="U$2" gate="G$1" x="121.92" y="5.08"/>
-<instance part="LOGO1" gate="G$1" x="121.92" y="20.32"/>
-<instance part="U$3" gate="G$1" x="121.92" y="5.08"/>
+<instance part="LOGO1" gate="G$1" x="170.18" y="45.72"/>
 <instance part="JP5" gate="G$1" x="236.22" y="25.4"/>
 <instance part="JP7" gate="G$1" x="233.68" y="25.4"/>
 <instance part="JP8" gate="G$1" x="243.84" y="27.94"/>
 <instance part="JP9" gate="G$1" x="243.84" y="25.4"/>
+<instance part="LOGO2" gate="G$1" x="187.96" y="38.1"/>
+<instance part="LOGO4" gate="G$1" x="148.59" y="7.366"/>
+<instance part="LOGO3" gate="G$1" x="186.69" y="38.608"/>
 </instances>
 <busses>
@@
 </segment>
 <segment>
-<pinref part="J2" gate="G$1" pin="VCC"/>
+<pinref part="J2" gate="G$1" pin="2"/>
 <wire x1="43.18" y1="45.72" x2="40.64" y2="45.72" width="0.1524" layer="91"/>
 <wire x1="40.64" y1="45.72" x2="40.64" y2="53.34" width="0.1524" layer="91"/>
@@
 </segment>
 <segment>
-<pinref part="J4" gate="G$1" pin="VCC"/>
+<pinref part="J4" gate="G$1" pin="2"/>
 <wire x1="43.18" y1="17.78" x2="40.64" y2="17.78" width="0.1524" layer="91"/>
 <wire x1="40.64" y1="17.78" x2="40.64" y2="25.4" width="0.1524" layer="91"/>
@@
 </segment>
 <segment>
-<pinref part="J2" gate="G$1" pin="GND"/>
+<pinref part="J2" gate="G$1" pin="1"/>
 <wire x1="43.18" y1="43.18" x2="40.64" y2="43.18" width="0.1524" layer="91"/>
 <wire x1="40.64" y1="43.18" x2="40.64" y2="40.64" width="0.1524" layer="91"/>
@@
 </segment>
 <segment>
-<pinref part="J4" gate="G$1" pin="GND"/>
+<pinref part="J4" gate="G$1" pin="1"/>
 <wire x1="43.18" y1="15.24" x2="40.64" y2="15.24" width="0.1524" layer="91"/>
 <wire x1="40.64" y1="15.24" x2="40.64" y2="12.7" width="0.1524" layer="91"/>
@@
 <net name="SCL" class="0">
 <segment>
-<pinref part="J2" gate="G$1" pin="SCL"/>
+<pinref part="J2" gate="G$1" pin="4"/>
 <wire x1="43.18" y1="50.8" x2="38.1" y2="50.8" width="0.1524" layer="91"/>
 <label x="38.1" y="50.8" size="1.27" layer="95" rot="R180" xref="yes"/>
@@
 </segment>
 <segment>
-<pinref part="J4" gate="G$1" pin="SCL"/>
+<pinref part="J4" gate="G$1" pin="4"/>
 <wire x1="43.18" y1="22.86" x2="38.1" y2="22.86" width="0.1524" layer="91"/>
 <label x="38.1" y="22.86" size="1.27" layer="95" rot="R180" xref="yes"/>
@@
 <net name="SDA" class="0">
 <segment>
-<pinref part="J2" gate="G$1" pin="SDA"/>
+<pinref part="J2" gate="G$1" pin="3"/>
 <wire x1="43.18" y1="48.26" x2="38.1" y2="48.26" width="0.1524" layer="91"/>
 <label x="38.1" y="48.26" size="1.27" layer="95" rot="R180" xref="yes"/>
@@
 </segment>
 <segment>
-<pinref part="J4" gate="G$1" pin="SDA"/>
+<pinref part="J4" gate="G$1" pin="3"/>
 <wire x1="43.18" y1="20.32" x2="38.1" y2="20.32" width="0.1524" layer="91"/>
 <label x="38.1" y="20.32" size="1.27" layer="95" rot="R180" xref="yes"/>

Commit message: Post design review changes
Other:
- note added: "Cut trace on jumper JP1 to remove I2C pullups"
- note added: "This is the 110 Degree FOV version of the board, there is also a board, SEN-14844, with a 55 Degree FOV"
- note added: "VIN: 3-3.6V"
- note added: "v10"
- note removed: "v01"
Changed lines of the file:
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@@
 <?xml version="1.0" encoding="utf-8"?>
 <!DOCTYPE eagle SYSTEM "eagle.dtd">
-<eagle version="9.0.1">
+<eagle version="9.1.0">
 <drawing>
 <settings>
@@
 <plain>
 <text x="76.708" y="101.346" size="1.778" layer="97">Power</text>
-<text x="165.354" y="11.43" size="2.54" layer="94">Jim Lindblom</text>
-<text x="106.68" y="93.98" size="1.778" layer="97">7-bit unshifted I2C Address: 0x33</text>
-<text x="236.22" y="7.62" size="2.54" layer="94" font="vector">v01</text>
+<text x="165.354" y="11.43" size="2.54" layer="94" font="vector">Jim Lindblom</text>
+<text x="106.68" y="93.98" size="1.778" layer="97" font="vector">7-bit unshifted I2C Address: 0x33</text>
+<text x="236.22" y="7.62" size="2.54" layer="94" font="vector">v10</text>
 <text x="168.656" y="7.366" size="2.54" layer="94" font="vector">Andy England</text>
 <text x="114.3" y="132.08" size="2.54" layer="95" font="vector">MLX90640</text>
 <text x="50.8" y="63.5" size="2.54" layer="95" font="vector">Qwiic/I2C Conections</text>
+<wire x1="0" y1="81.28" x2="248.92" y2="81.28" width="0.1524" layer="97" style="longdash"/>
+<text x="114.3" y="129.54" size="1.778" layer="97" font="vector">VIN: 3-3.6V</text>
+<text x="10.16" y="2.54" size="1.778" layer="97" font="vector">This is the 110 Degree FOV version of the board, there is also a board, SEN-14844, with a 55 Degree FOV</text>
+<text x="175.26" y="124.46" size="1.778" layer="97" font="vector">Cut trace on jumper JP1 to remove I2C pullups</text>
 </plain>
 <instances>
@@
 <pinref part="J2" gate="G$1" pin="4"/>
 <wire x1="43.18" y1="50.8" x2="38.1" y2="50.8" width="0.1524" layer="91"/>
-<label x="38.1" y="50.8" size="1.27" layer="95" rot="R180" xref="yes"/>
+<label x="38.1" y="50.8" size="1.27" layer="95" font="vector" rot="R180" xref="yes"/>
 </segment>
 <segment>
 <pinref part="J3" gate="G$1" pin="SCL"/>
 <wire x1="76.2" y1="50.8" x2="71.12" y2="50.8" width="0.1524" layer="91"/>
-<label x="71.12" y="50.8" size="1.27" layer="95" rot="R180" xref="yes"/>
+<label x="71.12" y="50.8" size="1.27" layer="95" font="vector" rot="R180" xref="yes"/>
 </segment>
 <segment>
 <pinref part="J4" gate="G$1" pin="4"/>
 <wire x1="43.18" y1="22.86" x2="38.1" y2="22.86" width="0.1524" layer="91"/>
-<label x="38.1" y="22.86" size="1.27" layer="95" rot="R180" xref="yes"/>
+<label x="38.1" y="22.86" size="1.27" layer="95" font="vector" rot="R180" xref="yes"/>
 </segment>
 <segment>
 <pinref part="U1" gate="G$1" pin="SCL"/>
 <wire x1="134.62" y1="106.68" x2="137.16" y2="106.68" width="0.1524" layer="91"/>
-<label x="137.16" y="106.68" size="1.27" layer="95" xref="yes"/>
+<label x="137.16" y="106.68" size="1.27" layer="95" font="vector" xref="yes"/>
 </segment>
 <segment>
@@
 <wire x1="180.34" y1="106.68" x2="180.34" y2="101.6" width="0.1524" layer="91"/>
 <wire x1="180.34" y1="101.6" x2="162.56" y2="101.6" width="0.1524" layer="91"/>
-<label x="162.56" y="101.6" size="1.27" layer="95" rot="R180" xref="yes"/>
+<label x="162.56" y="101.6" size="1.27" layer="95" font="vector" rot="R180" xref="yes"/>
 </segment>
 </net>
@@
 <pinref part="J2" gate="G$1" pin="3"/>
 <wire x1="43.18" y1="48.26" x2="38.1" y2="48.26" width="0.1524" layer="91"/>
-<label x="38.1" y="48.26" size="1.27" layer="95" rot="R180" xref="yes"/>
+<label x="38.1" y="48.26" size="1.27" layer="95" font="vector" rot="R180" xref="yes"/>
 </segment>
 <segment>
 <pinref part="J3" gate="G$1" pin="SDA"/>
 <wire x1="76.2" y1="48.26" x2="71.12" y2="48.26" width="0.1524" layer="91"/>
-<label x="71.12" y="48.26" size="1.27" layer="95" rot="R180" xref="yes"/>
+<label x="71.12" y="48.26" size="1.27" layer="95" font="vector" rot="R180" xref="yes"/>
 </segment>
 <segment>
 <pinref part="J4" gate="G$1" pin="3"/>
 <wire x1="43.18" y1="20.32" x2="38.1" y2="20.32" width="0.1524" layer="91"/>
-<label x="38.1" y="20.32" size="1.27" layer="95" rot="R180" xref="yes"/>
+<label x="38.1" y="20.32" size="1.27" layer="95" font="vector" rot="R180" xref="yes"/>
 </segment>
 <segment>
 <pinref part="U1" gate="G$1" pin="SDA"/>
 <wire x1="134.62" y1="111.76" x2="137.16" y2="111.76" width="0.1524" layer="91"/>
-<label x="137.16" y="111.76" size="1.27" layer="95" xref="yes"/>
+<label x="137.16" y="111.76" size="1.27" layer="95" font="vector" xref="yes"/>
 </segment>
 <segment>
@@
 <wire x1="165.1" y1="106.68" x2="165.1" y2="104.14" width="0.1524" layer="91"/>
 <wire x1="162.56" y1="104.14" x2="165.1" y2="104.14" width="0.1524" layer="91"/>
-<label x="162.56" y="104.14" size="1.27" layer="95" rot="R180" xref="yes"/>
+<label x="162.56" y="104.14" size="1.27" layer="95" font="vector" rot="R180" xref="yes"/>
 </segment>
 </net>

Commit message: fixing issues
Changed lines of the file:
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@@
 <wire x1="0" y1="81.28" x2="248.92" y2="81.28" width="0.1524" layer="97" style="longdash"/>
 <text x="114.3" y="129.54" size="1.778" layer="97" font="vector">VIN: 3-3.6V</text>
-<text x="10.16" y="2.54" size="1.778" layer="97" font="vector">This is the 110 Degree FOV version of the board, there is also a board, SEN-14844, with a 55 Degree FOV</text>
+<text x="60.96" y="86.36" size="1.778" layer="97" font="vector">This is the 110 Degree FOV version of the board, there is also a board, SEN-14844, with a 55 Degree FOV</text>
 <text x="175.26" y="124.46" size="1.778" layer="97" font="vector">Cut trace on jumper JP1 to remove I2C pullups</text>
 </plain>
